File: Project/IDB_remaster.kicad_pcb (KiCad board)
At the start: 2 copper layers, 282.6 x 104.5 mm, 155 parts, among them J1 AVR-ISP-6, K1 , K10 , K11 , K12 , K13 , K14 , K14_1 , K15 , K16 , K17 , K18 , K19 , K2 , K20 , K21 , K22 , K23 , K24 , K25 , K26 , K27 , K28 , K28_1 , K29 , K29_1 , K3 , K30 , K31 , K32 , K33 , K34 , K35 , K36 , K37 , K38 , K39 , K4 , K40 , K41 , K41_1 , K42 , K43 , K43_1 , K44 , K45 , K46 , K47 , K48 , K49 , K5 , K50 , K51 , K52 , K53 , K54 , K55 , K55_1 , K56 , K57 , K58 , K59 , K6 , K60 , K61 , K62 , K63 , K7 , K8 , K9 , U1 PRTR5V0U2X, U2 ATmega32U4-AU, Y1 16mHz

Commit message: V1.3
Parts:
- removed the G*** at (93.3, 177.6)
- added G***: LOGO, Graphics:idb, F.Cu at (90.0, 178.2)
- RST: renamed from JP1; value RST -> JP1
- moved D28 0.27 mm to (256.5, 122.9)
- turned K28 to 0 degrees
Routing:
- net Net-(D28-Pad2): track 16.5 -> 31.1 mm
- net col13: track 213.8 -> 225.2 mm
- net row2: track 346.3 -> 345.8 mm
- net GND: vias 3 -> 4
Other:
- net class Default removed
- net class Power removed
- board text removed: "REMASTERED"
