File: Project/IDB_reborn.kicad_pcb (KiCad board)
At the start: 2 copper layers, 282.6 x 104.5 mm, 155 parts, among them J1 AVR-ISP-6, K1 , K10 , K11 , K12 , K13 , K14 , K14_1 , K15 , K16 , K17 , K18 , K19 , K2 , K20 , K21 , K22 , K23 , K24 , K25 , K26 , K27 , K28 , K28_1 , K29 , K29_1 , K3 , K30 , K31 , K32 , K33 , K34 , K35 , K36 , K37 , K38 , K39 , K4 , K40 , K41 , K41_1 , K42 , K43 , K43_1 , K44 , K45 , K46 , K47 , K48 , K49 , K5 , K50 , K51 , K52 , K53 , K54 , K55 , K55_1 , K56 , K57 , K58 , K59 , K6 , K60 , K61 , K62 , K63 , K7 , K8 , K9 , U1 PRTR5V0U2X, U2 ATmega32U4-AU, Y1 16mHz

Commit message: Final
Parts:
- moved D28 3.73 mm to (253.5, 120.7), turned to 90 degrees
Routing:
- net Net-(D28-Pad2): track 31.1 -> 34.6 mm
- net row1: track 311.3 -> 310.2 mm
Changed lines of the file:
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@@
       (effects (font (size 1.524 1.524) (thickness 0.3)))
     )
-    (fp_text user locked "REMASTER" (at 22 5.5 unlocked) (layer "F.Mask")
+    (fp_text user locked "REBORN" (at 20 5.5 unlocked) (layer "F.Mask")
       (effects (font (size 3 3) (thickness 0.75)))
     )
@@
   )
   (footprint "random-keyboard-parts:D_SOD-123-Pretty" (layer "B.Cu")
-    (at 256.50108 122.90634)
+    (at 253.492 120.70825 90)
     (descr "SOD-123")
     (tags "SOD-123")
     (attr smd)
-    (fp_text reference "D28" (at -1.099 2.15325) (layer "B.SilkS")
+    (fp_text reference "D28" (at -1.099 2.15325 90) (layer "B.SilkS")
       (effects (font (size 1 1) (thickness 0.15)) (justify mirror))
     )
-    (fp_text value "D" (at 0 -2.1) (layer "B.Fab")
+    (fp_text value "D" (at 0 -2.1 90) (layer "B.Fab")
       (effects (font (size 1 1) (thickness 0.15)) (justify mirror))
     )
-    (fp_text user "${REFERENCE}" (at 0 2) (layer "B.Fab")
+    (fp_text user "${REFERENCE}" (at 0 2 90) (layer "B.Fab")
       (effects (font (size 1 1) (thickness 0.15)) (justify mirror))
     )
@@
     (fp_line (start -0.35 0) (end 0.25 0.4) (layer "B.Fab") (width 0.1))
     (fp_line (start -1.4 0.9) (end 1.4 0.9) (layer "B.Fab") (width 0.1))
-    (pad "1" smd rect locked (at -1.65 0) (size 0.9 1.2) (layers "B.Cu" "B.Paste" "B.Mask")
+    (pad "1" smd rect locked (at -1.65 0 90) (size 0.9 1.2) (layers "B.Cu" "B.Paste" "B.Mask")
       (net 3 "row1"))
-    (pad "2" smd rect locked (at 1.65 0) (size 0.9 1.2) (layers "B.Cu" "B.Paste" "B.Mask")
+    (pad "2" smd rect locked (at 1.65 0 90) (size 0.9 1.2) (layers "B.Cu" "B.Paste" "B.Mask")
       (net 32 "Net-(D28-Pad2)"))
     (model "${KISYS3DMOD}/Diode_SMD.3dshapes/D_SOD-123.step"
@@
   (segment (start 186.830049 122.829951) (end 187.36 122.3) (width 0.254) (layer "B.Cu") (net 3))
   (segment (start 75.678951 122.829951) (end 91.834049 122.829951) (width 0.254) (layer "B.Cu") (net 3))
+  (segment (start 252.35 122.35825) (end 251.80191 122.90634) (width 0.254) (layer "B.Cu") (net 3))
   (segment (start 208.647951 122.829951) (end 224.803049 122.829951) (width 0.254) (layer "B.Cu") (net 3))
   (segment (start 54.264 122.3) (end 55.118 122.3) (width 0.254) (layer "B.Cu") (net 3))
+  (segment (start 246.69734 122.90634) (end 246.091 122.3) (width 0.254) (layer "B.Cu") (net 3))
   (segment (start 189.597951 122.829951) (end 205.880049 122.829951) (width 0.254) (layer "B.Cu") (net 3))
   (segment (start 148.857049 122.829951) (end 149.387 122.3) (width 0.254) (layer "B.Cu") (net 3))
@@
   (segment (start 132.045 122.3) (end 132.574951 122.829951) (width 0.254) (layer "B.Cu") (net 3))
   (segment (start 226.187 122.3) (end 227.041 122.3) (width 0.254) (layer "B.Cu") (net 3))
-  (segment (start 246.091 122.3) (end 246.453355 122.662355) (width 0.254) (layer "B.Cu") (net 3))
   (segment (start 34.60975 123.03125) (end 35.341 122.3) (width 0.254) (layer "B.Cu") (net 3))
-  (segment (start 246.69734 122.90634) (end 246.453355 122.662355) (width 0.254) (layer "B.Cu") (net 3))
   (segment (start 170.777701 122.829951) (end 186.830049 122.829951) (width 0.254) (layer "B.Cu") (net 3))
   (segment (start 129.807049 122.829951) (end 130.337 122.3) (width 0.254) (layer "B.Cu") (net 3))
@@
   (segment (start 165.331827 171.022424) (end 163.980318 171.022424) (width 0.254) (layer "B.Cu") (net 3))
   (segment (start 168.437 122.3) (end 169.291 122.3) (width 0.254) (layer "B.Cu") (net 3))
+  (segment (start 253.492 122.35825) (end 252.35 122.35825) (width 0.254) (layer "B.Cu") (net 3))
+  (segment (start 246.091 122.3) (end 245.237 122.3) (width 0.254) (layer "B.Cu") (net 3))
   (segment (start 227.570951 122.829951) (end 243.853049 122.829951) (width 0.254) (layer "B.Cu") (net 3))
   (segment (start 13.427 122.3) (end 14.15825 123.03125) (width 0.254) (layer "B.Cu") (net 3))
@@
   (segment (start 74.295 122.3) (end 75.149 122.3) (width 0.254) (layer "B.Cu") (net 3))
   (segment (start 169.832168 171.94006) (end 170.602989 171.169239) (width 0.254) (layer "B.Cu") (net 3))
+  (segment (start 251.80191 122.90634) (end 246.69734 122.90634) (width 0.254) (layer "B.Cu") (net 3))
   (segment (start 170.942 126.42325) (end 170.942 122.99425) (width 0.254) (layer "B.Cu") (net 3))
   (segment (start 37.049 122.3) (end 37.78025 123.03125) (width 0.254) (layer "B.Cu") (net 3))
@@
   (segment (start 187.36 122.3) (end 188.214 122.3) (width 0.254) (layer "B.Cu") (net 3))
   (segment (start 243.853049 122.829951) (end 244.383 122.3) (width 0.254) (layer "B.Cu") (net 3))
-  (segment (start 254.85108 122.90634) (end 246.69734 122.90634) (width 0.254) (layer "B.Cu") (net 3))
   (segment (start 188.214 122.3) (end 189.068 122.3) (width 0.254) (layer "B.Cu") (net 3))
   (segment (start 113.651951 122.829951) (end 129.807049 122.829951) (width 0.254) (layer "B.Cu") (net 3))
@@
   (segment (start 12.573 122.3) (end 13.427 122.3) (width 0.254) (layer "B.Cu") (net 3))
   (segment (start 130.337 122.3) (end 131.191 122.3) (width 0.254) (layer "B.Cu") (net 3))
-  (segment (start 245.237 122.3) (end 246.091 122.3) (width 0.254) (layer "B.Cu") (net 3))
   (segment (start 55.972 122.3) (end 56.672 123) (width 0.254) (layer "B.Cu") (net 3))
   (segment (start 167.386 171.94006) (end 166.249462 171.94006) (width 0.254) (layer "B.Cu") (net 3))
@@
   (segment (start 240.04 115.45125) (end 243.58875 119) (width 0.254) (layer "B.Cu") (net 31))
   (segment (start 243.58875 119) (end 245.237 119) (width 0.254) (layer "B.Cu") (net 31))
-  (segment (start 268.705 130.98026) (end 264.58943 126.86469) (width 0.254) (layer "B.Cu") (net 32))
-  (segment (start 268.705 130.98026) (end 268.705 132.57125) (width 0.254) (layer "B.Cu") (net 32))
-  (segment (start 263.79 122.74245) (end 263.62611 122.90634) (width 0.254) (layer "B.Cu") (net 32))
-  (segment (start 263.62611 122.90634) (end 258.87609 122.90634) (width 0.254) (layer "B.Cu") (net 32))
+  (segment (start 263.79 115.45125) (end 263.79 122.34825) (width 0.254) (layer "B.Cu") (net 32))
   (segment (start 262.04277 126.07302) (end 262.83444 126.86469) (width 0.254) (layer "B.Cu") (net 32))
-  (segment (start 258.87609 122.90634) (end 262.04277 126.07302) (width 0.254) (layer "B.Cu") (net 32))
-  (segment (start 263.79 115.45125) (end 263.79 122.74245) (width 0.254) (layer "B.Cu") (net 32))
+  (segment (start 263.79 122.74245) (end 263.62611 122.90634) (width 0.254) (layer "B.Cu") (net 32))
   (segment (start 262.83444 126.86469) (end 264.58943 126.86469) (width 0.254) (layer "B.Cu") (net 32))
-  (segment (start 259.66776 123.69801) (end 262.04277 126.07302) (width 0.254) (layer "B.Cu") (net 32))
-  (segment (start 258.15108 122.90634) (end 258.87609 122.90634) (width 0.254) (layer "B.Cu") (net 32))
+  (segment (start 268.705 130.98026) (end 268.705 132.57125) (width 0.254) (layer "B.Cu") (net 32))
+  (segment (start 263.79 122.34825) (end 262.04277 124.09548) (width 0.254) (layer "B.Cu") (net 32))
+  (segment (start 253.492 117.40625) (end 253.492 119.05825) (width 0.254) (layer "B.Cu") (net 32))
+  (segment (start 262.04277 124.09548) (end 262.04277 126.07302) (width 0.254) (layer "B.Cu") (net 32))
+  (segment (start 255.447 115.45125) (end 253.492 117.40625) (width 0.254) (layer "B.Cu") (net 32))
+  (segment (start 263.79 115.45125) (end 255.447 115.45125) (width 0.254) (layer "B.Cu") (net 32))
+  (segment (start 264.58943 126.86469) (end 268.705 130.98026) (width 0.254) (layer "B.Cu") (net 32))
   (segment (start 172.045988 172.01224) (end 172.045988 164.738238) (width 0.254) (layer "F.Cu") (net 33))
   (segment (start 171.745989 172.312239) (end 172.045988 172.01224) (width 0.254) (layer "F.Cu") (net 33))
